Commit message: Wheels rotating, cleanup todo, robot not moving

File: urdf/robot.urdf (robot description, URDF)
Before this commit: robot omni_wheel_base, 4 links, 3 joints
Joints:
- joint wheel_1_joint: axis (none) -> 0 0 1
- joint wheel_2_joint: axis 0 1 0 -> 0 0 1
- joint wheel_3_joint: axis 0 1 0 -> 0 0 1
